Commit message: Correcting URDF File

File: src/four_drive_mecanum_robot_description/urdf/four_drive_mecanum_robot.xacro (robot description, xacro)
@@ -6,6 +6,6 @@
 <link name="base_link">
   <inertial>
-    <origin xyz="0.1565398920687127 -0.004788955871560701 0.030358758115536476" rpy="0 0 0"/>
-    <mass value="43.71464533998368"/>
+    <origin xyz="0.006039892215173973 -0.004788955871560998 0.020358758115537435" rpy="0 0 0"/>
+    <mass value="43.71464533998373"/>
     <inertia ixx="1.998681" iyy="0.98793" izz="2.531812" ixy="-0.008367" iyz="-0.003455" ixz="-0.003863"/>
   </inertial>
@@ -26,10 +26,10 @@
 <link name="front_left_wheel_1">
   <inertial>
-    <origin xyz="0.042583798412730745 -1.4339203141533474e-07 3.450111268538114e-06" rpy="0 0 0"/>
+    <origin xyz="0.04258379844209284 -1.4339203130431244e-07 3.4501112685658697e-06" rpy="0 0 0"/>
     <mass value="6.195492949588099"/>
     <inertia ixx="0.039964" iyy="0.022937" izz="0.022937" ixy="-0.0" iyz="-0.0" ixz="1e-06"/>
   </inertial>
   <visual>
-    <origin xyz="-0.345938 0.254962 0.053172" rpy="0 0 0"/>
+    <origin xyz="-0.195438 0.254962 0.063172" rpy="0 0 0"/>
     <geometry>
       <mesh filename="file://$(find four_drive_mecanum_robot_description)/meshes/front_left_wheel_1.stl" scale="0.001 0.001 0.001"/>
@@ -38,5 +38,5 @@
   </visual>
   <collision>
-    <origin xyz="-0.345938 0.254962 0.053172" rpy="0 0 0"/>
+    <origin xyz="-0.195438 0.254962 0.063172" rpy="0 0 0"/>
     <geometry>
       <mesh filename="file://$(find four_drive_mecanum_robot_description)/meshes/front_left_wheel_1.stl" scale="0.001 0.001 0.001"/>
@@ -46,10 +46,10 @@
 <link name="lidar_1">
   <inertial>
-    <origin xyz="-4.4262982168419285e-11 -3.428023143126069e-11 0.012500303766958043" rpy="0 0 0"/>
-    <mass value="0.6512177959195155"/>
-    <inertia ixx="0.000206" iyy="0.000206" izz="0.000344" ixy="-0.0" iyz="0.0" ixz="0.0"/>
+    <origin xyz="-1.4900243365534305e-11 -3.427629360897022e-11 0.012500303766958015" rpy="0 0 0"/>
+    <mass value="0.6512177959195157"/>
+    <inertia ixx="0.000206" iyy="0.000206" izz="0.000344" ixy="0.0" iyz="0.0" ixz="0.0"/>
   </inertial>
   <visual>
-    <origin xyz="-0.1495 0.009 -0.181125" rpy="0 0 0"/>
+    <origin xyz="0.001 0.009 -0.171125" rpy="0 0 0"/>
     <geometry>
       <mesh filename="file://$(find four_drive_mecanum_robot_description)/meshes/lidar_1.stl" scale="0.001 0.001 0.001"/>
@@ -58,5 +58,5 @@
   </visual>
   <collision>
-    <origin xyz="-0.1495 0.009 -0.181125" rpy="0 0 0"/>
+    <origin xyz="0.001 0.009 -0.171125" rpy="0 0 0"/>
     <geometry>
       <mesh filename="file://$(find four_drive_mecanum_robot_description)/meshes/lidar_1.stl" scale="0.001 0.001 0.001"/>
@@ -66,10 +66,10 @@
 <link name="camera_link_1">
   <inertial>
-    <origin xyz="-0.04750630918678708 -0.015024630338028797 1.256722554077161e-07" rpy="0 0 0"/>
-    <mass value="0.8360165625360608"/>
-    <inertia ixx="0.000122" iyy="0.001047" izz="0.001049" ixy="0.0" iyz="-0.0" ixz="0.0"/>
+    <origin xyz="-0.04726155287090634 -0.015030443332914215 0.007574813766801719" rpy="0 0 0"/>
+    <mass value="0.6763864753348693"/>
+    <inertia ixx="8.6e-05" iyy="0.000761" izz="0.000776" ixy="0.0" iyz="0.0" ixz="-2e-06"/>
   </inertial>
   <visual>
-    <origin xyz="-0.198 0.074 -0.174407" rpy="0 0 0"/>
+    <origin xyz="-0.047 0.074 -0.154407" rpy="0 0 0"/>
     <geometry>
       <mesh filename="file://$(find four_drive_mecanum_robot_description)/meshes/camera_link_1.stl" scale="0.001 0.001 0.001"/>
@@ -78,5 +78,5 @@
   </visual>
   <collision>
-    <origin xyz="-0.198 0.074 -0.174407" rpy="0 0 0"/>
+    <origin xyz="-0.047 0.074 -0.154407" rpy="0 0 0"/>
     <geometry>
       <mesh filename="file://$(find four_drive_mecanum_robot_description)/meshes/camera_link_1.stl" scale="0.001 0.001 0.001"/>
@@ -86,10 +86,10 @@
 <link name="front_right_wheel_1">
   <inertial>
-    <origin xyz="-0.04258379847145508 -1.4339203141533474e-07 3.450111268801792e-06" rpy="0 0 0"/>
+    <origin xyz="-0.04258379844209309 -1.433920313598236e-07 3.45011126881567e-06" rpy="0 0 0"/>
     <mass value="6.1954929495881"/>
     <inertia ixx="0.039964" iyy="0.022937" izz="0.022937" ixy="0.0" iyz="-0.0" ixz="-1e-06"/>
   </inertial>
   <visual>
-    <origin xyz="0.044938 0.254962 0.053172" rpy="0 0 0"/>
+    <origin xyz="0.195438 0.254962 0.063172" rpy="0 0 0"/>
     <geometry>
       <mesh filename="file://$(find four_drive_mecanum_robot_description)/meshes/front_right_wheel_1.stl" scale="0.001 0.001 0.001"/>
@@ -98,5 +98,5 @@
   </visual>
   <collision>
-    <origin xyz="0.044938 0.254962 0.053172" rpy="0 0 0"/>
+    <origin xyz="0.195438 0.254962 0.063172" rpy="0 0 0"/>
     <geometry>
       <mesh filename="file://$(find four_drive_mecanum_robot_description)/meshes/front_right_wheel_1.stl" scale="0.001 0.001 0.001"/>
@@ -106,10 +106,10 @@
 <link name="rear_left_wheel_1">
   <inertial>
-    <origin xyz="0.042583798412730745 1.4339203141533474e-07 3.4501112687046476e-06" rpy="0 0 0"/>
+    <origin xyz="0.04258379844209281 1.4339203063817862e-07 3.450111268732403e-06" rpy="0 0 0"/>
     <mass value="6.1954929495881"/>
     <inertia ixx="0.039964" iyy="0.022937" izz="0.022937" ixy="0.0" iyz="0.0" ixz="1e-06"/>
   </inertial>
   <visual>
-    <origin xyz="-0.345938 -0.254962 0.053172" rpy="0 0 0"/>
+    <origin xyz="-0.195438 -0.254962 0.063172" rpy="0 0 0"/>
     <geometry>
       <mesh filename="file://$(find four_drive_mecanum_robot_description)/meshes/rear_left_wheel_1.stl" scale="0.001 0.001 0.001"/>
@@ -118,5 +118,5 @@
   </visual>
   <collision>
-    <origin xyz="-0.345938 -0.254962 0.053172" rpy="0 0 0"/>
+    <origin xyz="-0.195438 -0.254962 0.063172" rpy="0 0 0"/>
     <geometry>
       <mesh filename="file://$(find four_drive_mecanum_robot_description)/meshes/rear_left_wheel_1.stl" scale="0.001 0.001 0.001"/>
@@ -126,10 +126,10 @@
 <link name="rear_right_wheel_1">
   <inertial>
-    <origin xyz="-0.04258379847145511 1.4339203141533474e-07 3.4501112686421975e-06" rpy="0 0 0"/>
+    <origin xyz="-0.04258379844209309 1.4339203063817862e-07 3.4501112686491364e-06" rpy="0 0 0"/>
     <mass value="6.195492949588099"/>
     <inertia ixx="0.039964" iyy="0.022937" izz="0.022937" ixy="-0.0" iyz="0.0" ixz="-1e-06"/>
   </inertial>
   <visual>
-    <origin xyz="0.044938 -0.254962 0.053172" rpy="0 0 0"/>
+    <origin xyz="0.195438 -0.254962 0.063172" rpy="0 0 0"/>
     <geometry>
       <mesh filename="file://$(find four_drive_mecanum_robot_description)/meshes/rear_right_wheel_1.stl" scale="0.001 0.001 0.001"/>
@@ -138,5 +138,5 @@
   </visual>
   <collision>
-    <origin xyz="0.044938 -0.254962 0.053172" rpy="0 0 0"/>
+    <origin xyz="0.195438 -0.254962 0.063172" rpy="0 0 0"/>
     <geometry>
       <mesh filename="file://$(find four_drive_mecanum_robot_description)/meshes/rear_right_wheel_1.stl" scale="0.001 0.001 0.001"/>
@@ -145,5 +145,5 @@
 </link>
 <joint name="front_left_joint" type="continuous">
-  <origin xyz="0.345938 -0.254962 -0.053172" rpy="0 0 0"/>
+  <origin xyz="0.195438 -0.254962 -0.063172" rpy="0 0 0"/>
   <parent link="base_link"/>
   <child link="front_left_wheel_1"/>
@@ -151,5 +151,5 @@
 </joint>
 <joint name="lidar_joint" type="continuous">
-  <origin xyz="0.1495 -0.009 0.181125" rpy="0 0 0"/>
+  <origin xyz="-0.001 -0.009 0.171125" rpy="0 0 0"/>
   <parent link="base_link"/>
   <child link="lidar_1"/>
@@ -157,10 +157,10 @@
 </joint>
 <joint name="camera_joint" type="fixed">
-  <origin xyz="0.198 -0.074 0.174407" rpy="0 0 0"/>
+  <origin xyz="0.047 -0.074 0.154407" rpy="0 0 0"/>
   <parent link="base_link"/>
   <child link="camera_link_1"/>
 </joint>
 <joint name="front_right_joint" type="continuous">
-  <origin xyz="-0.044938 -0.254962 -0.053172" rpy="0 0 0"/>
+  <origin xyz="-0.195438 -0.254962 -0.063172" rpy="0 0 0"/>
   <parent link="base_link"/>
   <child link="front_right_wheel_1"/>
@@ -168,5 +168,5 @@
 </joint>
 <joint name="rear_left_joint" type="continuous">
-  <origin xyz="0.345938 0.254962 -0.053172" rpy="0 0 0"/>
+  <origin xyz="0.195438 0.254962 -0.063172" rpy="0 0 0"/>
   <parent link="base_link"/>
   <child link="rear_left_wheel_1"/>
@@ -174,5 +174,5 @@
 </joint>
 <joint name="rear_right_joint" type="continuous">
-  <origin xyz="-0.044938 0.254962 -0.053172" rpy="0 0 0"/>
+  <origin xyz="-0.195438 0.254962 -0.063172" rpy="0 0 0"/>
   <parent link="base_link"/>
   <child link="rear_right_wheel_1"/>

Commit message: Updated the URDF of the robot

File: src/four_drive_mecanum_robot_description/urdf/four_drive_mecanum_robot.xacro (robot description, xacro)
@@ -2,11 +2,10 @@
 <robot name="four_drive_mecanum_robot" xmlns:xacro="http://www.ros.org/wiki/xacro">
 <xacro:include filename="$(find four_drive_mecanum_robot_description)/urdf/materials.xacro" />
-<xacro:include filename="$(find four_drive_mecanum_robot_description)/urdf/four_drive_mecanum_robot.trans" />
 <xacro:include filename="$(find four_drive_mecanum_robot_description)/urdf/four_drive_mecanum_robot.gazebo" />
 <link name="base_link">
   <inertial>
-    <origin xyz="0.006039892215173973 -0.004788955871560998 0.020358758115537435" rpy="0 0 0"/>
-    <mass value="43.71464533998373"/>
-    <inertia ixx="1.998681" iyy="0.98793" izz="2.531812" ixy="-0.008367" iyz="-0.003455" ixz="-0.003863"/>
+    <origin xyz="0.004788955754076288 0.006039892215565465 0.02035875811553353" rpy="0 0 0"/>
+    <mass value="43.71464533998358"/>
+    <inertia ixx="0.98793" iyy="1.998681" izz="2.531812" ixy="0.008367" iyz="-0.003863" ixz="0.003455"/>
   </inertial>
   <visual>
@@ -26,10 +25,10 @@
 <link name="front_left_wheel_1">
   <inertial>
-    <origin xyz="0.04258379844209284 -1.4339203130431244e-07 3.4501112685658697e-06" rpy="0 0 0"/>
+    <origin xyz="1.4339193726842225e-07 0.04258379844209284 -2.5970406986319805e-06" rpy="0 0 0"/>
     <mass value="6.195492949588099"/>
-    <inertia ixx="0.039964" iyy="0.022937" izz="0.022937" ixy="-0.0" iyz="-0.0" ixz="1e-06"/>
+    <inertia ixx="0.022937" iyy="0.039964" izz="0.022937" ixy="-0.0" iyz="-1e-06" ixz="0.0"/>
   </inertial>
   <visual>
-    <origin xyz="-0.195438 0.254962 0.063172" rpy="0 0 0"/>
+    <origin xyz="-0.254962 -0.195438 0.063172" rpy="0 0 0"/>
     <geometry>
       <mesh filename="file://$(find four_drive_mecanum_robot_description)/meshes/front_left_wheel_1.stl" scale="0.001 0.001 0.001"/>
@@ -38,5 +37,5 @@
   </visual>
   <collision>
-    <origin xyz="-0.195438 0.254962 0.063172" rpy="0 0 0"/>
+    <origin xyz="-0.254962 -0.195438 0.063172" rpy="0 0 0"/>
     <geometry>
       <mesh filename="file://$(find four_drive_mecanum_robot_description)/meshes/front_left_wheel_1.stl" scale="0.001 0.001 0.001"/>
@@ -44,12 +43,72 @@
   </collision>
 </link>
+<link name="front_right_wheel_1">
+  <inertial>
+    <origin xyz="1.433919372129111e-07 -0.042583798442092785 -2.5970406988123917e-06" rpy="0 0 0"/>
+    <mass value="6.1954929495881"/>
+    <inertia ixx="0.022937" iyy="0.039964" izz="0.022937" ixy="0.0" iyz="1e-06" ixz="0.0"/>
+  </inertial>
+  <visual>
+    <origin xyz="-0.254962 0.195438 0.063172" rpy="0 0 0"/>
+    <geometry>
+      <mesh filename="file://$(find four_drive_mecanum_robot_description)/meshes/front_right_wheel_1.stl" scale="0.001 0.001 0.001"/>
+    </geometry>
+    <material name="silver"/>
+  </visual>
+  <collision>
+    <origin xyz="-0.254962 0.195438 0.063172" rpy="0 0 0"/>
+    <geometry>
+      <mesh filename="file://$(find four_drive_mecanum_robot_description)/meshes/front_right_wheel_1.stl" scale="0.001 0.001 0.001"/>
+    </geometry>
+  </collision>
+</link>
+<link name="rear_left_wheel_1">
+  <inertial>
+    <origin xyz="-1.433919372129111e-07 0.042583798442092785 -2.5970406988123917e-06" rpy="0 0 0"/>
+    <mass value="6.1954929495881"/>
+    <inertia ixx="0.022937" iyy="0.039964" izz="0.022937" ixy="0.0" iyz="-1e-06" ixz="-0.0"/>
+  </inertial>
+  <visual>
+    <origin xyz="0.254962 -0.195438 0.063172" rpy="0 0 0"/>
+    <geometry>
+      <mesh filename="file://$(find four_drive_mecanum_robot_description)/meshes/rear_left_wheel_1.stl" scale="0.001 0.001 0.001"/>
+    </geometry>
+    <material name="silver"/>
+  </visual>
+  <collision>
+    <origin xyz="0.254962 -0.195438 0.063172" rpy="0 0 0"/>
+    <geometry>
+      <mesh filename="file://$(find four_drive_mecanum_robot_description)/meshes/rear_left_wheel_1.stl" scale="0.001 0.001 0.001"/>
+    </geometry>
+  </collision>
+</link>
+<link name="rear_right_wheel_1">
+  <inertial>
+    <origin xyz="-1.4339193726842225e-07 -0.04258379844209284 -2.5970406986319805e-06" rpy="0 0 0"/>
+    <mass value="6.195492949588099"/>
+    <inertia ixx="0.022937" iyy="0.039964" izz="0.022937" ixy="-0.0" iyz="1e-06" ixz="-0.0"/>
+  </inertial>
+  <visual>
+    <origin xyz="0.254962 0.195438 0.063172" rpy="0 0 0"/>
+    <geometry>
+      <mesh filename="file://$(find four_drive_mecanum_robot_description)/meshes/rear_right_wheel_1.stl" scale="0.001 0.001 0.001"/>
+    </geometry>
+    <material name="silver"/>
+  </visual>
+  <collision>
+    <origin xyz="0.254962 0.195438 0.063172" rpy="0 0 0"/>
+    <geometry>
+      <mesh filename="file://$(find four_drive_mecanum_robot_description)/meshes/rear_right_wheel_1.stl" scale="0.001 0.001 0.001"/>
+    </geometry>
+  </collision>
+</link>
 <link name="lidar_1">
   <inertial>
-    <origin xyz="-1.4900243365534305e-11 -3.427629360897022e-11 0.012500303766958015" rpy="0 0 0"/>
-    <mass value="0.6512177959195157"/>
-    <inertia ixx="0.000206" iyy="0.000206" izz="0.000344" ixy="0.0" iyz="0.0" ixz="0.0"/>
+    <origin xyz="3.4280042346401807e-11 -1.4901005776501997e-11 0.015000303766958017" rpy="0 0 0"/>
+    <mass value="0.7814613551034187"/>
+    <inertia ixx="0.000265" iyy="0.000265" izz="0.000413" ixy="-0.0" iyz="0.0" ixz="-0.0"/>
   </inertial>
   <visual>
-    <origin xyz="0.001 0.009 -0.171125" rpy="0 0 0"/>
+    <origin xyz="-0.009 0.001 -0.171125" rpy="0 0 0"/>
     <geometry>
       <mesh filename="file://$(find four_drive_mecanum_robot_description)/meshes/lidar_1.stl" scale="0.001 0.001 0.001"/>
@@ -58,5 +117,5 @@
   </visual>
   <collision>
-    <origin xyz="0.001 0.009 -0.171125" rpy="0 0 0"/>
+    <origin xyz="-0.009 0.001 -0.171125" rpy="0 0 0"/>
     <geometry>
       <mesh filename="file://$(find four_drive_mecanum_robot_description)/meshes/lidar_1.stl" scale="0.001 0.001 0.001"/>
@@ -66,10 +125,10 @@
 <link name="camera_link_1">
   <inertial>
-    <origin xyz="-0.04726155287090634 -0.015030443332914215 0.007574813766801719" rpy="0 0 0"/>
-    <mass value="0.6763864753348693"/>
-    <inertia ixx="8.6e-05" iyy="0.000761" izz="0.000776" ixy="0.0" iyz="0.0" ixz="-2e-06"/>
+    <origin xyz="0.00951620811188017 -0.047500004005499835 1.0139224432270666e-07" rpy="0 0 0"/>
+    <mass value="0.5293613918364843"/>
+    <inertia ixx="0.000662" iyy="5.4e-05" izz="0.000641" ixy="-0.0" iyz="0.0" ixz="0.0"/>
   </inertial>
   <visual>
-    <origin xyz="-0.047 0.074 -0.154407" rpy="0 0 0"/>
+    <origin xyz="-0.074 -0.0475 -0.164407" rpy="0 0 0"/>
     <geometry>
       <mesh filename="file://$(find four_drive_mecanum_robot_description)/meshes/camera_link_1.stl" scale="0.001 0.001 0.001"/>
@@ -78,5 +137,5 @@
   </visual>
   <collision>
-    <origin xyz="-0.047 0.074 -0.154407" rpy="0 0 0"/>
+    <origin xyz="-0.074 -0.0475 -0.164407" rpy="0 0 0"/>
     <geometry>
       <mesh filename="file://$(find four_drive_mecanum_robot_description)/meshes/camera_link_1.stl" scale="0.001 0.001 0.001"/>
@@ -84,72 +143,30 @@
   </collision>
 </link>
-<link name="front_right_wheel_1">
-  <inertial>
-    <origin xyz="-0.04258379844209309 -1.433920313598236e-07 3.45011126881567e-06" rpy="0 0 0"/>
-    <mass value="6.1954929495881"/>
-    <inertia ixx="0.039964" iyy="0.022937" izz="0.022937" ixy="0.0" iyz="-0.0" ixz="-1e-06"/>
-  </inertial>
-  <visual>
-    <origin xyz="0.195438 0.254962 0.063172" rpy="0 0 0"/>
-    <geometry>
-      <mesh filename="file://$(find four_drive_mecanum_robot_description)/meshes/front_right_wheel_1.stl" scale="0.001 0.001 0.001"/>
-    </geometry>
-    <material name="silver"/>
-  </visual>
-  <collision>
-    <origin xyz="0.195438 0.254962 0.063172" rpy="0 0 0"/>
-    <geometry>
-      <mesh filename="file://$(find four_drive_mecanum_robot_description)/meshes/front_right_wheel_1.stl" scale="0.001 0.001 0.001"/>
-    </geometry>
-  </collision>
-</link>
-<link name="rear_left_wheel_1">
-  <inertial>
-    <origin xyz="0.04258379844209281 1.4339203063817862e-07 3.450111268732403e-06" rpy="0 0 0"/>
-    <mass value="6.1954929495881"/>
-    <inertia ixx="0.039964" iyy="0.022937" izz="0.022937" ixy="0.0" iyz="0.0" ixz="1e-06"/>
-  </inertial>
-  <visual>
-    <origin xyz="-0.195438 -0.254962 0.063172" rpy="0 0 0"/>
-    <geometry>
-      <mesh filename="file://$(find four_drive_mecanum_robot_description)/meshes/rear_left_wheel_1.stl" scale="0.001 0.001 0.001"/>
-    </geometry>
-    <material name="silver"/>
-  </visual>
-  <collision>
-    <origin xyz="-0.195438 -0.254962 0.063172" rpy="0 0 0"/>
-    <geometry>
-      <mesh filename="file://$(find four_drive_mecanum_robot_description)/meshes/rear_left_wheel_1.stl" scale="0.001 0.001 0.001"/>
-    </geometry>
-  </collision>
-</link>
-<link name="rear_right_wheel_1">
-  <inertial>
-    <origin xyz="-0.04258379844209309 1.4339203063817862e-07 3.4501112686491364e-06" rpy="0 0 0"/>
-    <mass value="6.195492949588099"/>
-    <inertia ixx="0.039964" iyy="0.022937" izz="0.022937" ixy="-0.0" iyz="0.0" ixz="-1e-06"/>
-  </inertial>
-  <visual>
-    <origin xyz="0.195438 -0.254962 0.063172" rpy="0 0 0"/>
-    <geometry>
-      <mesh filename="file://$(find four_drive_mecanum_robot_description)/meshes/rear_right_wheel_1.stl" scale="0.001 0.001 0.001"/>
-    </geometry>
-    <material name="silver"/>
-  </visual>
-  <collision>
-    <origin xyz="0.195438 -0.254962 0.063172" rpy="0 0 0"/>
-    <geometry>
-      <mesh filename="file://$(find four_drive_mecanum_robot_description)/meshes/rear_right_wheel_1.stl" scale="0.001 0.001 0.001"/>
-    </geometry>
-  </collision>
-</link>
 <joint name="front_left_joint" type="continuous">
-  <origin xyz="0.195438 -0.254962 -0.063172" rpy="0 0 0"/>
+  <origin xyz="0.254962 0.195438 -0.063172" rpy="0 0 0"/>
   <parent link="base_link"/>
   <child link="front_left_wheel_1"/>
-  <axis xyz="1.0 0.0 0.0"/>
+  <axis xyz="0.0 1.0 0.0"/>
+</joint>
+<joint name="front_right_joint" type="continuous">
+  <origin xyz="0.254962 -0.195438 -0.063172" rpy="0 0 0"/>
+  <parent link="base_link"/>
+  <child link="front_right_wheel_1"/>
+  <axis xyz="0.0 -1.0 0.0"/>
+</joint>
+<joint name="rear_left_joint" type="continuous">
+  <origin xyz="-0.254962 0.195438 -0.063172" rpy="0 0 0"/>
+  <parent link="base_link"/>
+  <child link="rear_left_wheel_1"/>
+  <axis xyz="0.0 1.0 0.0"/>
+</joint>
+<joint name="rear_right_joint" type="continuous">
+  <origin xyz="-0.254962 -0.195438 -0.063172" rpy="0 0 0"/>
+  <parent link="base_link"/>
+  <child link="rear_right_wheel_1"/>
+  <axis xyz="0.0 -1.0 0.0"/>
 </joint>
 <joint name="lidar_joint" type="continuous">
-  <origin xyz="-0.001 -0.009 0.171125" rpy="0 0 0"/>
+  <origin xyz="0.009 -0.001 0.171125" rpy="0 0 0"/>
   <parent link="base_link"/>
   <child link="lidar_1"/>
@@ -157,25 +174,7 @@
 </joint>
 <joint name="camera_joint" type="fixed">
-  <origin xyz="0.047 -0.074 0.154407" rpy="0 0 0"/>
+  <origin xyz="0.074 0.0475 0.164407" rpy="0 0 0"/>
   <parent link="base_link"/>
   <child link="camera_link_1"/>
 </joint>
-<joint name="front_right_joint" type="continuous">
-  <origin xyz="-0.195438 -0.254962 -0.063172" rpy="0 0 0"/>
-  <parent link="base_link"/>
-  <child link="front_right_wheel_1"/>
-  <axis xyz="-1.0 0.0 0.0"/>
-</joint>
-<joint name="rear_left_joint" type="continuous">
-  <origin xyz="0.195438 0.254962 -0.063172" rpy="0 0 0"/>
-  <parent link="base_link"/>
-  <child link="rear_left_wheel_1"/>
-  <axis xyz="1.0 0.0 0.0"/>
-</joint>
-<joint name="rear_right_joint" type="continuous">
-  <origin xyz="-0.195438 0.254962 -0.063172" rpy="0 0 0"/>
-  <parent link="base_link"/>
-  <child link="rear_right_wheel_1"/>
-  <axis xyz="-1.0 0.0 0.0"/>
-</joint>
 </robot>
