Commit message: Trying to integrate mecanum_drive_controller with the bot and added ROS2 Controller for activating it

File: src/four_drive_mecanum_robot_description/urdf/four_drive_mecanum_robot.xacro (robot description, xacro)
@@ -2,5 +2,5 @@
 <robot name="four_drive_mecanum_robot" xmlns:xacro="http://www.ros.org/wiki/xacro">
 <xacro:include filename="$(find four_drive_mecanum_robot_description)/urdf/materials.xacro" />
-<xacro:include filename="$(find four_drive_mecanum_robot_description)/urdf/four_drive_mecanum_robot.gazebo" />
+<xacro:include filename="$(find four_drive_mecanum_robot_description)/urdf/ros2_control.xacro" />
 <link name="base_link">
   <inertial>
@@ -14,5 +14,5 @@
       <mesh filename="file://$(find four_drive_mecanum_robot_description)/meshes/base_link.stl" scale="0.001 0.001 0.001"/>
     </geometry>
-    <material name="silver"/>
+    <material name="orange"/>
   </visual>
   <collision>
@@ -23,5 +23,5 @@
   </collision>
 </link>
-<link name="front_left_wheel_1">
+<link name="front_left_wheel">
   <inertial>
     <origin xyz="1.4339193726842225e-07 0.04258379844209284 -2.5970406986319805e-06" rpy="0 0 0"/>
@@ -32,5 +32,5 @@
     <origin xyz="-0.254962 -0.195438 0.063172" rpy="0 0 0"/>
     <geometry>
-      <mesh filename="file://$(find four_drive_mecanum_robot_description)/meshes/front_left_wheel_1.stl" scale="0.001 0.001 0.001"/>
+      <mesh filename="file://$(find four_drive_mecanum_robot_description)/meshes/front_left_wheel.stl" scale="0.001 0.001 0.001"/>
     </geometry>
     <material name="silver"/>
@@ -39,9 +39,9 @@
     <origin xyz="-0.254962 -0.195438 0.063172" rpy="0 0 0"/>
     <geometry>
-      <mesh filename="file://$(find four_drive_mecanum_robot_description)/meshes/front_left_wheel_1.stl" scale="0.001 0.001 0.001"/>
+      <mesh filename="file://$(find four_drive_mecanum_robot_description)/meshes/front_left_wheel.stl" scale="0.001 0.001 0.001"/>
     </geometry>
   </collision>
 </link>
-<link name="front_right_wheel_1">
+<link name="front_right_wheel">
   <inertial>
     <origin xyz="1.433919372129111e-07 -0.042583798442092785 -2.5970406988123917e-06" rpy="0 0 0"/>
@@ -52,5 +52,5 @@
     <origin xyz="-0.254962 0.195438 0.063172" rpy="0 0 0"/>
     <geometry>
-      <mesh filename="file://$(find four_drive_mecanum_robot_description)/meshes/front_right_wheel_1.stl" scale="0.001 0.001 0.001"/>
+      <mesh filename="file://$(find four_drive_mecanum_robot_description)/meshes/front_right_wheel.stl" scale="0.001 0.001 0.001"/>
     </geometry>
     <material name="silver"/>
@@ -59,9 +59,9 @@
     <origin xyz="-0.254962 0.195438 0.063172" rpy="0 0 0"/>
     <geometry>
-      <mesh filename="file://$(find four_drive_mecanum_robot_description)/meshes/front_right_wheel_1.stl" scale="0.001 0.001 0.001"/>
+      <mesh filename="file://$(find four_drive_mecanum_robot_description)/meshes/front_right_wheel.stl" scale="0.001 0.001 0.001"/>
     </geometry>
   </collision>
 </link>
-<link name="rear_left_wheel_1">
+<link name="rear_left_wheel">
   <inertial>
     <origin xyz="-1.433919372129111e-07 0.042583798442092785 -2.5970406988123917e-06" rpy="0 0 0"/>
@@ -72,5 +72,5 @@
     <origin xyz="0.254962 -0.195438 0.063172" rpy="0 0 0"/>
     <geometry>
-      <mesh filename="file://$(find four_drive_mecanum_robot_description)/meshes/rear_left_wheel_1.stl" scale="0.001 0.001 0.001"/>
+      <mesh filename="file://$(find four_drive_mecanum_robot_description)/meshes/rear_left_wheel.stl" scale="0.001 0.001 0.001"/>
     </geometry>
     <material name="silver"/>
@@ -79,9 +79,9 @@
     <origin xyz="0.254962 -0.195438 0.063172" rpy="0 0 0"/>
     <geometry>
-      <mesh filename="file://$(find four_drive_mecanum_robot_description)/meshes/rear_left_wheel_1.stl" scale="0.001 0.001 0.001"/>
+      <mesh filename="file://$(find four_drive_mecanum_robot_description)/meshes/rear_left_wheel.stl" scale="0.001 0.001 0.001"/>
     </geometry>
   </collision>
 </link>
-<link name="rear_right_wheel_1">
+<link name="rear_right_wheel">
   <inertial>
     <origin xyz="-1.4339193726842225e-07 -0.04258379844209284 -2.5970406986319805e-06" rpy="0 0 0"/>
@@ -92,5 +92,5 @@
     <origin xyz="0.254962 0.195438 0.063172" rpy="0 0 0"/>
     <geometry>
-      <mesh filename="file://$(find four_drive_mecanum_robot_description)/meshes/rear_right_wheel_1.stl" scale="0.001 0.001 0.001"/>
+      <mesh filename="file://$(find four_drive_mecanum_robot_description)/meshes/rear_right_wheel.stl" scale="0.001 0.001 0.001"/>
     </geometry>
     <material name="silver"/>
@@ -99,9 +99,9 @@
     <origin xyz="0.254962 0.195438 0.063172" rpy="0 0 0"/>
     <geometry>
-      <mesh filename="file://$(find four_drive_mecanum_robot_description)/meshes/rear_right_wheel_1.stl" scale="0.001 0.001 0.001"/>
+      <mesh filename="file://$(find four_drive_mecanum_robot_description)/meshes/rear_right_wheel.stl" scale="0.001 0.001 0.001"/>
     </geometry>
   </collision>
 </link>
-<link name="lidar_1">
+<link name="lidar">
   <inertial>
     <origin xyz="3.4280042346401807e-11 -1.4901005776501997e-11 0.015000303766958017" rpy="0 0 0"/>
@@ -112,16 +112,16 @@
     <origin xyz="-0.009 0.001 -0.171125" rpy="0 0 0"/>
     <geometry>
-      <mesh filename="file://$(find four_drive_mecanum_robot_description)/meshes/lidar_1.stl" scale="0.001 0.001 0.001"/>
+      <mesh filename="file://$(find four_drive_mecanum_robot_description)/meshes/lidar.stl" scale="0.001 0.001 0.001"/>
     </geometry>
-    <material name="silver"/>
+    <material name="black"/>
   </visual>
   <collision>
     <origin xyz="-0.009 0.001 -0.171125" rpy="0 0 0"/>
     <geometry>
-      <mesh filename="file://$(find four_drive_mecanum_robot_description)/meshes/lidar_1.stl" scale="0.001 0.001 0.001"/>
+      <mesh filename="file://$(find four_drive_mecanum_robot_description)/meshes/lidar.stl" scale="0.001 0.001 0.001"/>
     </geometry>
   </collision>
 </link>
-<link name="camera_link_1">
+<link name="camera_link">
   <inertial>
     <origin xyz="0.00951620811188017 -0.047500004005499835 1.0139224432270666e-07" rpy="0 0 0"/>
@@ -132,12 +132,12 @@
     <origin xyz="-0.074 -0.0475 -0.164407" rpy="0 0 0"/>
     <geometry>
-      <mesh filename="file://$(find four_drive_mecanum_robot_description)/meshes/camera_link_1.stl" scale="0.001 0.001 0.001"/>
+      <mesh filename="file://$(find four_drive_mecanum_robot_description)/meshes/camera_link.stl" scale="0.001 0.001 0.001"/>
     </geometry>
-    <material name="silver"/>
+    <material name="black"/>
   </visual>
   <collision>
     <origin xyz="-0.074 -0.0475 -0.164407" rpy="0 0 0"/>
     <geometry>
-      <mesh filename="file://$(find four_drive_mecanum_robot_description)/meshes/camera_link_1.stl" scale="0.001 0.001 0.001"/>
+      <mesh filename="file://$(find four_drive_mecanum_robot_description)/meshes/camera_link.stl" scale="0.001 0.001 0.001"/>
     </geometry>
   </collision>
@@ -146,5 +146,5 @@
   <origin xyz="0.254962 0.195438 -0.063172" rpy="0 0 0"/>
   <parent link="base_link"/>
-  <child link="front_left_wheel_1"/>
+  <child link="front_left_wheel"/>
   <axis xyz="0.0 1.0 0.0"/>
 </joint>
@@ -152,11 +152,11 @@
   <origin xyz="0.254962 -0.195438 -0.063172" rpy="0 0 0"/>
   <parent link="base_link"/>
-  <child link="front_right_wheel_1"/>
-  <axis xyz="0.0 -1.0 0.0"/>
+  <child link="front_right_wheel"/>
+  <axis xyz="0.0 1.0 0.0"/>
 </joint>
 <joint name="rear_left_joint" type="continuous">
   <origin xyz="-0.254962 0.195438 -0.063172" rpy="0 0 0"/>
   <parent link="base_link"/>
-  <child link="rear_left_wheel_1"/>
+  <child link="rear_left_wheel"/>
   <axis xyz="0.0 1.0 0.0"/>
 </joint>
@@ -164,11 +164,11 @@
   <origin xyz="-0.254962 -0.195438 -0.063172" rpy="0 0 0"/>
   <parent link="base_link"/>
-  <child link="rear_right_wheel_1"/>
-  <axis xyz="0.0 -1.0 0.0"/>
+  <child link="rear_right_wheel"/>
+  <axis xyz="0.0 1.0 0.0"/>
 </joint>
 <joint name="lidar_joint" type="continuous">
   <origin xyz="0.009 -0.001 0.171125" rpy="0 0 0"/>
   <parent link="base_link"/>
-  <child link="lidar_1"/>
+  <child link="lidar"/>
   <axis xyz="0.0 0.0 1.0"/>
 </joint>
@@ -176,5 +176,5 @@
   <origin xyz="0.074 0.0475 0.164407" rpy="0 0 0"/>
   <parent link="base_link"/>
-  <child link="camera_link_1"/>
+  <child link="camera_link"/>
 </joint>
 </robot>

File: src/four_drive_mecanum_robot_description/urdf/materials.xacro (robot description, xacro)
@@ -1,6 +1,12 @@
 <?xml version="1.0" ?>
 <robot name="four_drive_mecanum_robot" xmlns:xacro="http://www.ros.org/wiki/xacro" >
-<material name="silver">
-  <color rgba="0.700 0.700 0.700 1.000"/>
-</material>
+  <material name="silver">
+    <color rgba="0.7 0.7 0.7 1.0"/>
+  </material>
+  <material name="orange">
+    <color rgba="1 0.3 0.1 1"/>
+  </material>
+  <material name="black">
+    <color rgba="0.0 0.0 0.0 1.0"/>
+  </material>
 </robot>

Commit message: Added gazebo planar move plugin and performed Visual SLAM

File: src/four_drive_mecanum_robot_description/urdf/four_drive_mecanum_robot.xacro (robot description, xacro)
@@ -2,5 +2,7 @@
 <robot name="four_drive_mecanum_robot" xmlns:xacro="http://www.ros.org/wiki/xacro">
 <xacro:include filename="$(find four_drive_mecanum_robot_description)/urdf/materials.xacro" />
-<xacro:include filename="$(find four_drive_mecanum_robot_description)/urdf/ros2_control.xacro" />
+<xacro:include filename="$(find four_drive_mecanum_robot_description)/urdf/gazebo.xacro" />
+<!-- <xacro:include filename="$(find four_drive_mecanum_robot_description)/urdf/ros2_control.xacro" /> -->
+<xacro:property name="PI" value="3.1415926535897931"/>
 <link name="base_link">
   <inertial>
@@ -37,7 +39,8 @@
   </visual>
   <collision>
-    <origin xyz="-0.254962 -0.195438 0.063172" rpy="0 0 0"/>
+    <origin xyz="0 0.04 0" rpy="${PI/2} 0 0"/>
     <geometry>
-      <mesh filename="file://$(find four_drive_mecanum_robot_description)/meshes/front_left_wheel.stl" scale="0.001 0.001 0.001"/>
+      <!-- <mesh filename="file://$(find four_drive_mecanum_robot_description)/meshes/front_left_wheel.stl" scale="0.001 0.001 0.001"/> -->
+      <cylinder radius="0.103" length="0.07798"/>
     </geometry>
   </collision>
@@ -57,7 +60,8 @@
   </visual>
   <collision>
-    <origin xyz="-0.254962 0.195438 0.063172" rpy="0 0 0"/>
+    <origin xyz="0 -0.04 0" rpy="${PI/2} 0 0"/>
     <geometry>
-      <mesh filename="file://$(find four_drive_mecanum_robot_description)/meshes/front_right_wheel.stl" scale="0.001 0.001 0.001"/>
+      <!-- <mesh filename="file://$(find four_drive_mecanum_robot_description)/meshes/front_left_wheel.stl" scale="0.001 0.001 0.001"/> -->
+      <cylinder radius="0.103" length="0.07798"/>
     </geometry>
   </collision>
@@ -77,7 +81,8 @@
   </visual>
   <collision>
-    <origin xyz="0.254962 -0.195438 0.063172" rpy="0 0 0"/>
+    <origin xyz="0 0.04 0" rpy="${PI/2} 0 0"/>
     <geometry>
-      <mesh filename="file://$(find four_drive_mecanum_robot_description)/meshes/rear_left_wheel.stl" scale="0.001 0.001 0.001"/>
+      <!-- <mesh filename="file://$(find four_drive_mecanum_robot_description)/meshes/front_left_wheel.stl" scale="0.001 0.001 0.001"/> -->
+      <cylinder radius="0.103" length="0.07798"/>
     </geometry>
   </collision>
@@ -97,7 +102,8 @@
   </visual>
   <collision>
-    <origin xyz="0.254962 0.195438 0.063172" rpy="0 0 0"/>
+    <origin xyz="0 -0.04 0" rpy="${PI/2} 0 0"/>
     <geometry>
-      <mesh filename="file://$(find four_drive_mecanum_robot_description)/meshes/rear_right_wheel.stl" scale="0.001 0.001 0.001"/>
+      <!-- <mesh filename="file://$(find four_drive_mecanum_robot_description)/meshes/front_left_wheel.stl" scale="0.001 0.001 0.001"/> -->
+      <cylinder radius="0.103" length="0.07798"/>
     </geometry>
   </collision>
@@ -143,4 +149,10 @@
   </collision>
 </link>
+<joint name="camera_optical_joint" type="fixed">
+  <parent link="camera_link"/>
+  <child link="camera_color_frame"/>
+  <origin xyz="0.03 -0.0475 0.0" rpy="${-pi/2} 0 ${-pi/2}"/>
+</joint>
+<link name="camera_color_frame"></link>
 <joint name="front_left_joint" type="continuous">
   <origin xyz="0.254962 0.195438 -0.063172" rpy="0 0 0"/>
@@ -167,5 +179,5 @@
   <axis xyz="0.0 1.0 0.0"/>
 </joint>
-<joint name="lidar_joint" type="continuous">
+<joint name="lidar_joint" type="fixed">
   <origin xyz="0.009 -0.001 0.171125" rpy="0 0 0"/>
   <parent link="base_link"/>

File: src/four_drive_mecanum_robot_description/urdf/gazebo.xacro (robot description, xacro)
@@ -5,65 +5,102 @@
   <xacro:property name="sensor_color" value="Gazebo/Black" />
   <gazebo>
-    <plugin name="diff_drive" filename="libgazebo_ros_diff_drive.so">
-      <num_wheel_pairs>2</num_wheel_pairs>
-      <left_joint>front_left_joint</left_joint>
-      <right_joint>front_right_joint</right_joint>
-      <left_joint>rear_left_joint</left_joint>
-      <right_joint>rear_right_joint</right_joint>
-      <wheel_separation>0.259</wheel_separation>
-      <wheel_separation>0.259</wheel_separation>
-      <wheel_diameter>0.203</wheel_diameter>
-      <wheel_diameter>0.203</wheel_diameter>
-      <max_wheel_torque>200</max_wheel_torque>
-      <max_wheel_acceleration>10.0</max_wheel_acceleration>
+    <plugin name="mecanum_drive" filename="libgazebo_ros_planar_move.so">
+      <command_topic>cmd_vel</command_topic>
+      <odometry_topic>odom</odometry_topic>
       <odometry_frame>odom</odometry_frame>
+      <odometry_rate>20.0</odometry_rate>
       <robot_base_frame>base_link</robot_base_frame>
       <publish_odom>true</publish_odom>
       <publish_odom_tf>true</publish_odom_tf>
-      <publish_wheel_tf>true</publish_wheel_tf>
     </plugin>
   </gazebo>
-<gazebo reference="base_link">
-  <material>${body_color}</material>
-  <mu1>0.2</mu1>
-  <mu2>0.2</mu2>
-  <self_collide>true</self_collide>
-  <gravity>true</gravity>
-</gazebo>
-<gazebo reference="front_left_wheel">
-  <material>${wheel_color}</material>
-  <mu1>0.2</mu1>
-  <mu2>0.2</mu2>
-  <self_collide>true</self_collide>
-</gazebo>
-<gazebo reference="front_right_wheel">
-  <material>${wheel_color}</material>
-  <mu1>0.2</mu1>
-  <mu2>0.2</mu2>
-  <self_collide>true</self_collide>
-</gazebo>
-<gazebo reference="rear_left_wheel">
-  <material>${wheel_color}</material>
-  <mu1>0.2</mu1>
-  <mu2>0.2</mu2>
-  <self_collide>true</self_collide>
-</gazebo>
-<gazebo reference="rear_right_wheel">
-  <material>${wheel_color}</material>
-  <mu1>0.2</mu1>
-  <mu2>0.2</mu2>
-  <self_collide>true</self_collide>
-</gazebo>
-<gazebo reference="lidar">
-  <material>${sensor_color}</material>
-  <mu1>0.2</mu1>
-  <mu2>0.2</mu2>
-  <self_collide>true</self_collide>
-</gazebo>
-<gazebo reference="camera_link">
-  <material>${sensor_color}</material>
-  <mu1>0.2</mu1>
-  <mu2>0.2</mu2>
-  <self_collide>true</self_collide>
-</gazebo>
+  <gazebo reference="lidar">
+    <material>${sensor_color}</material>
+    <sensor name="laser" type="ray">
+      <pose> 0 0 0 0 0 0 </pose>
+      <visualize>true</visualize>
+      <update_rate>10</update_rate>
+      <ray>
+        <scan>
+          <horizontal>
+            <samples>360</samples>
+            <min_angle>-3.14</min_angle>
+            <max_angle>3.14</max_angle>
+          </horizontal>
+        </scan>
+      <range>
+        <min>0.3</min>
+        <max>12</max>
+      </range>
+      </ray>
+      <plugin name="laser_controller" filename="libgazebo_ros_ray_sensor.so">
+        <ros>
+            <remapping>/laser_controller/out:=/scan</remapping>
+        </ros>
+        <output_type>sensor_msgs/LaserScan</output_type>
+        <frame_name>lidar</frame_name>
+      </plugin>
+    </sensor>
+  </gazebo>
+  <!-- < This is the gazebo plugin for depth camera> -->
+  <gazebo reference="camera_link">
+    <sensor name="camera" type="depth">
+      <update_rate>20</update_rate>
+      <camera>
+        <horizontal_fov>1.012291</horizontal_fov>
+        <image>
+          <width>640</width>
+          <height>480</height>
+          <format>R8G8B8</format>
+        </image>
+        <clip>
+          <near>0.3</near>
+          <far>3</far>
+        </clip>
+      </camera>
+      <plugin name="camera_controller" filename="libgazebo_ros_camera.so">
+        <update_rate>1.0</update_rate>
+        <frame_name>camera_color_frame</frame_name>
+        <min_depth>0.1</min_depth>
+        <max_depth>100.0</max_depth>
+      </plugin>
+    </sensor>
+  </gazebo>
+  <gazebo reference="base_link">
+    <material>${body_color}</material>
+    <mu1>0.2</mu1>
+    <mu2>0.2</mu2>
+    <self_collide>true</self_collide>
+    <gravity>true</gravity>
+  </gazebo>
+  <gazebo reference="front_left_wheel">
+    <material>${wheel_color}</material>
+    <mu1>0.2</mu1>
+    <mu2>0.2</mu2>
+    <self_collide>true</self_collide>
+  </gazebo>
+  <gazebo reference="front_right_wheel">
+    <material>${wheel_color}</material>
+    <mu1>0.2</mu1>
+    <mu2>0.2</mu2>
+    <self_collide>true</self_collide>
+  </gazebo>
+  <gazebo reference="rear_left_wheel">
+    <material>${wheel_color}</material>
+    <mu1>0.2</mu1>
+    <mu2>0.2</mu2>
+    <self_collide>true</self_collide>
+  </gazebo>
+  <gazebo reference="rear_right_wheel">
+    <material>${wheel_color}</material>
+    <mu1>0.2</mu1>
+    <mu2>0.2</mu2>
+    <self_collide>true</self_collide>
+  </gazebo>
+  <gazebo reference="camera_link">
+    <material>${sensor_color}</material>
+    <mu1>0.2</mu1>
+    <mu2>0.2</mu2>
+    <self_collide>true</self_collide>
+  </gazebo>
 </robot>

Commit message: Added Nav2 plugin for the mecanum wheel and created a new world for Gazebo

File: src/four_drive_mecanum_robot_description/urdf/four_drive_mecanum_robot.xacro (robot description, xacro)
@@ -155,4 +155,5 @@
 </joint>
 <link name="camera_color_frame"></link>
+<link name="base_footprint"></link>
 <joint name="front_left_joint" type="continuous">
   <origin xyz="0.254962 0.195438 -0.063172" rpy="0 0 0"/>
@@ -190,3 +191,8 @@
   <child link="camera_link"/>
 </joint>
+<joint name="base_footprint_joint" type="fixed">
+  <origin xyz="0.0 0.0 -0.166" rpy="0 0 0"/>
+  <parent link="base_link"/>
+  <child link="base_footprint"/>
+</joint>
 </robot>

File: src/four_drive_mecanum_robot_description/urdf/gazebo.xacro (robot description, xacro)
@@ -46,4 +46,5 @@
   <gazebo reference="camera_link">
     <sensor name="camera" type="depth">
+      <visualize>true</visualize>
       <update_rate>20</update_rate>
       <camera>
@@ -56,5 +57,5 @@
         <clip>
           <near>0.3</near>
-          <far>3</far>
+          <far>6</far>
         </clip>
       </camera>
